Commit message: added pendulum

File: examples/pybullet/gym/pybullet_data/inverted_double_pendulum.urdf (robot description, URDF)
Before this commit: robot , 5 links, 4 joints
Links:
- removed link link1_1
- removed link link1_2
- removed link link1_4
- added link link2_1, mass 0.00000
- added link link2_2, mass 0.00000
- added link link2_4, mass 0.00000
- added link link2_6, mass 0.00000
- added link pole2, mass 4.19874; collision capsule length=0.60000 radius=0.04500
- link pole: mass 5.01859 -> 4.19874; geometry collision capsule length=0.60000 radius=0.04500
Joints:
- removed joint jointfix_0_4
- removed joint jointfix_1_2
- added joint hinge2: type continuous, parent pole, child link2_6, origin xyz=0.00000 0.00000 0.60000 rpy=0.00000 -0.00000 0.00000, axis 0.00000 1.00000 0.00000
- added joint jointfix_0_6: type fixed, parent link2_6, child pole2, origin xyz=0.00000 0.00000 0.00000 rpy=0.00000 -0.00000 0.00000, axis 0.00000 0.00000 0.00000
- added joint jointfix_1_4: type fixed, parent link2_4, child pole, origin xyz=0.00000 0.00000 0.00000 rpy=0.00000 -0.00000 0.00000, axis 0.00000 0.00000 0.00000
- added joint jointfix_2_2: type fixed, parent link2_2, child cart, origin xyz=0.00000 0.00000 0.00000 rpy=0.00000 -0.00000 0.00000, axis 0.00000 0.00000 0.00000
- joint hinge: child link1_4 -> link2_4
- joint slider: child link1_2 -> link2_2; parent link1_1 -> link2_1
