Commit message: default pd for pybullet, 100, 1 for physx

File: examples/pybullet/gym/pybullet_data/ant_torso.urdf (robot description, URDF)
Before this commit: robot ant, 21 links, 20 joints
Links:
- link front_left_foot: geometry collision capsule length=0.56569 radius=0.08000; visual capsule length=0.56569 radius=0.08000
- link front_left_leg: geometry collision capsule length=0.28284 radius=0.08000; visual capsule length=0.28284 radius=0.08000
- link front_right_foot: geometry collision capsule length=0.56569 radius=0.08000; visual capsule length=0.56569 radius=0.08000
- link front_right_leg: geometry collision capsule length=0.28284 radius=0.08000; visual capsule length=0.28284 radius=0.08000
- link left_back_foot: geometry collision capsule length=0.56569 radius=0.08000; visual capsule length=0.56569 radius=0.08000
- link left_back_leg: geometry collision capsule length=0.28284 radius=0.08000; visual capsule length=0.28284 radius=0.08000
- link right_back_foot: geometry collision capsule length=0.56569 radius=0.08000; visual capsule length=0.56569 radius=0.08000
- link right_back_leg: geometry collision capsule length=0.28284 radius=0.08000; visual capsule length=0.28284 radius=0.08000
