Commit message: torso is root link now

File: examples/pybullet/gym/pybullet_data/half_cheetah.urdf (robot description, URDF)
Before this commit: robot cheetah, 17 links, 16 joints
Links:
- removed link link0_1
- removed link link0_2
- removed link link0_3
- removed link link0_4
- added link link1, mass 0.00000
- added link link2, mass 0.00000
- added link link3, mass 0.00000
Joints:
- removed joint jointfix_6_4
- joint ignorex: child link0_2 -> link1; parent link0_1 -> torso
- joint ignorey: child link0_4 -> link3; parent link0_3 -> torso
- joint ignorez: child link0_3 -> link2; parent link0_2 -> torso
