Commit message: 2d versions work now

File: examples/pybullet/gym/pybullet_data/hopper.urdf (robot description, URDF)
Before this commit: robot hopper, 11 links, 10 joints
Links:
- removed link link0_4
Joints:
- removed joint jointfix_3_4
- joint ignore1: child link0_2 -> link0_1; parent link0_1 -> torso
- joint ignore2: child link0_3 -> link0_2; parent link0_2 -> torso
- joint ignore3: child link0_4 -> link0_3; parent link0_3 -> torso

File: examples/pybullet/gym/pybullet_data/walker2d.urdf (robot description, URDF)
Before this commit: robot walker2d, 17 links, 16 joints
Links:
- removed link link0_4
Joints:
- removed joint jointfix_6_4
- joint ignorex: child link0_2 -> link0_1; parent link0_1 -> torso
- joint ignorey: child link0_4 -> link0_3; parent link0_3 -> torso
- joint ignorez: child link0_3 -> link0_2; parent link0_2 -> torso
